File: kicad/keytar/keytar.kicad_pcb (KiCad board)
At the start: 2 copper layers, 70 x 90 mm, 38 parts, among them J1 , J2 USB_B, J3 AudioJack2, J4 Conn_01x04, J5 USB_A, J6 Mini-DIN-6-Shielded, J7 Conn_01x04, Q1 BSS138, Q2 BSS138, U1 Pico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

Commit message: improve pcb
Parts:
- added J_NO_BATT1: Jumper_2_Open, Jumper:SolderJumper-2_P1.3mm_Open_RoundedPad1.0x1.5mm, F.Cu at (142.9, 141.5)
- added SW1: SW_DPST_x2, Connector_JST:JST_XH_B3B-XH-A_1x03_P2.50mm_Vertical, F.Cu at (155.0, 142.0)
- REF** (x4): value MountingHole_3.2mm_M3 -> MountingHole_3.2mm_M3_ISO14580_Pad; footprint MountingHole:MountingHole_3.2mm_M3 -> MountingHole:MountingHole_3.2mm_M3_ISO14580_Pad
- U1: footprint MCU_RaspberryPi_and_Boards:RPi_Pico_SMD_TH -> keyar-parts:RPi_Pico_debug_hole_USB_SMD_TH
- moved C3 2.55 mm to (139.1, 138.0)
- moved D1 2.55 mm to (145.8, 135.4)
- moved L1 2.55 mm to (150.3, 131.1)
- moved R10 2.55 mm to (139.2, 130.2)
- moved R11 2.55 mm to (139.2, 134.2)
- moved U3 2.55 mm to (145.0, 131.1)
- moved REF** 1.41 mm to (124.0, 141.0)
- moved REF** 1.41 mm to (186.0, 141.0)
- moved REF** 1.41 mm to (124.0, 59.0)
- moved REF** 1.41 mm to (186.0, 59.0)
- moved D3 1.00 mm to (174.7, 60.0)
- moved D2 0.83 mm to (174.7, 82.5)
Connections:
- net Net-(D1-A) renamed /REG_OUT
- net Net-(SW1A-B) renamed /REG_IN
- net USB D+ renamed USB HOST D+
- net USB D- renamed USB HOST D-
- J2 pad 2: unconnected-(J2-D--Pad2) -> USB DEV D-
- J2 pad 3: unconnected-(J2-D+-Pad3) -> USB DEV D+
- J2 pad 5: unconnected-(J2-Shield-Pad5) -> GND
Routing:
- net USB DEV D-: track 0.00 -> 49.6 mm
- net USB DEV D+: track 0.00 -> 49.3 mm
- net +5V: track 102.3 -> 125.1 mm
- net /REG_IN: track 4.28 -> 23.0 mm
- net +BATT: track 16.7 -> 32.9 mm
- net VBUS: track 102.2 -> 113.5 mm, vias 0 -> 2
- net GND: track 5.54 -> 12.2 mm, vias 2 -> 3
- net +3V3: track 127.3 -> 132.6 mm, vias 1 -> 2
- net Net-(D3-A): track 11.3 -> 10.3 mm
- net Net-(U1-GPIO26_ADC0): track 43.7 -> 44.6 mm, vias 0 -> 1
- net Net-(D2-A): track 5.48 -> 4.65 mm
Other:
- outline, holes or cut-outs redrawn
- board text added: "Analog"
- board text added: "Battery management"
- board text added: "I²C"
- board text added: "MIDI out"
- board text added: "PS/2"
- board text added: "Pedal"
- board text added: "Pico"
- board text added: "USB device"
- board text added: "USB host"
